Commit message: Update: Improve code portability and documentation

File: src/ros2_kortex/kortex_description/robots/gen3_2f85.urdf (robot description, URDF)
Before this commit: robot gen3_, 30 links, 29 joints
Links:
- link gen3_base_link: geometry collision mesh filename=package://kortex_description/arms/gen3/7dof/meshes/base_lin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; visual mesh filename=package://kortex_description/arms/gen3/7dof/meshes/base_lin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
- link gen3_bracelet_link: geometry collision mesh filename=package://kortex_description/arms/gen3/7dof/meshes/bracelet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; visual mesh filename=package://kortex_description/arms/gen3/7dof/meshes/bracelet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
- link gen3_forearm_link: geometry collision mesh filename=package://kortex_description/arms/gen3/7dof/meshes/forearm_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; visual mesh filename=package://kortex_description/arms/gen3/7dof/meshes/forearm_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
- link gen3_half_arm_1_link: geometry collision mesh filename=package://kortex_description/arms/gen3/7dof/meshes/half_arm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; visual mesh filename=package://kortex_description/arms/gen3/7dof/meshes/half_arm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
- link gen3_half_arm_2_link: geometry collision mesh filename=package://kortex_description/arms/gen3/7dof/meshes/half_arm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; visual mesh filename=package://kortex_description/arms/gen3/7dof/meshes/half_arm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
- link gen3_robotiq_85_base_link: geometry collision mesh filename=package://robotiq_description/meshes/collision/robotiq_base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; visual mesh filename=package://robotiq_description/meshes/visual/robotiq_base.dae
- link gen3_robotiq_85_left_finger_link: geometry collision mesh filename=package://robotiq_description/meshes/collision/left_finger.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; visual mesh filename=package://robotiq_description/meshes/visual/left_finger.dae
- link gen3_robotiq_85_left_finger_tip_link: geometry collision mesh filename=package://robotiq_description/meshes/collision/left_finger_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; visual mesh filename=package://robotiq_description/meshes/visual/left_finger_tip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
- link gen3_robotiq_85_left_inner_knuckle_link: geometry collision mesh filename=package://robotiq_description/meshes/collision/left_inner_k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; visual mesh filename=package://robotiq_description/meshes/visual/left_inner_knuc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
- link gen3_robotiq_85_left_knuckle_link: geometry collision mesh filename=package://robotiq_description/meshes/collision/left_knuckle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; visual mesh filename=package://robotiq_description/meshes/visual/left_knuckle.dae
- link gen3_robotiq_85_right_finger_link: geometry collision mesh filename=package://robotiq_description/meshes/collision/right_finger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; visual mesh filename=package://robotiq_description/meshes/visual/right_finger.dae
- link gen3_robotiq_85_right_finger_tip_link: geometry collision mesh filename=package://robotiq_description/meshes/collision/right_finger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; visual mesh filename=package://robotiq_description/meshes/visual/right_finger_ti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
- link gen3_robotiq_85_right_inner_knuckle_link: geometry collision mesh filename=package://robotiq_description/meshes/collision/right_inner_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; visual mesh filename=package://robotiq_description/meshes/visual/right_inner_knu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
- link gen3_robotiq_85_right_knuckle_link: geometry collision mesh filename=package://robotiq_description/meshes/collision/right_knuckl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; visual mesh filename=package://robotiq_description/meshes/visual/right_knuckle.d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
- link gen3_shoulder_link: geometry collision mesh filename=package://kortex_description/arms/gen3/7dof/meshes/shoulder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; visual mesh filename=package://kortex_description/arms/gen3/7dof/meshes/shoulder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
- link gen3_spherical_wrist_1_link: geometry collision mesh filename=package://kortex_description/arms/gen3/7dof/meshes/spherica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; visual mesh filename=package://kortex_description/arms/gen3/7dof/meshes/spherica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
- link gen3_spherical_wrist_2_link: geometry collision mesh filename=package://kortex_description/arms/gen3/7dof/meshes/spherica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; visual mesh filename=package://kortex_description/arms/gen3/7dof/meshes/spherica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
- link wrist_mounted_camera_link: geometry collision box size=0.02505 0.090 0.025; visual mesh filename=package://realsense2_description/meshes/d435.dae
