Commit message: 增加了机械臂在gazebo里

File: install/kortex_description/share/kortex_description/robots/kinova.urdf.xacro (robot description, xacro)
@@ -1,141 +1,144 @@
 <?xml version="1.0"?>
-<robot xmlns:xacro="http://ros.org/wiki/xacro" name="$(arg name)">
+<robot xmlns:xacro="http://ros.org/wiki/xacro">
+  <!-- Define the robot name argument before using it -->
+  <xacro:arg name="name" default="kinova_arm" />
   <!-- robot name parameter -->
-  <xacro:arg name="name" default="kinova_arm" />
-  <!-- Arguments -->
-  <xacro:arg name="prefix" default="" />
-  <xacro:arg name="arm" default="NO_ARM_TYPE_DEFINED" />
-  <xacro:arg name="dof" default="7" />
-  <xacro:arg name="vision" default="false" />
-  <xacro:arg name="robot_ip" default="192.168.11.11" />
-  <xacro:arg name="username" default="admin" />
-  <xacro:arg name="password" default="admin" />
-  <xacro:arg name="port" default="10000" />
-  <xacro:arg name="port_realtime" default="10001" />
-  <xacro:arg name="session_inactivity_timeout_ms" default="60000" />
-  <xacro:arg name="connection_inactivity_timeout_ms" default="2000" />
-  <xacro:arg name="gripper" default="" />
-  <xacro:arg name="gripper_joint_name" default="finger_joint" />
-  <xacro:arg name="gripper_max_velocity" default="100.0" />
-  <xacro:arg name="gripper_max_force" default="100.0" />
-  <xacro:arg name="use_internal_bus_gripper_comm" default="false" />
-  <xacro:arg name="use_fake_hardware" default="false" />
-  <xacro:arg name="fake_sensor_commands" default="false" />
-  <xacro:arg name="sim_gazebo" default="false" />
-  <xacro:arg name="sim_isaac" default="false" />
-  <xacro:arg name="gazebo_renderer" default="ogre"/>
-  <xacro:arg name="camera_width" default="640"/>
-  <xacro:arg name="camera_height" default="480"/>
-  <xacro:arg name="camera_fps" default="6"/>
-  <xacro:arg name="simulation_controllers" default="$(find kortex_description)/arm/$(arg arm)/$(arg dof)dof/config/ros2_controllers.yaml" />
-  <xacro:arg name="moveit_active" default="false"/>
-  <!-- import main macro -->
-  <xacro:include filename="$(find kortex_description)/robots/kortex_robot.xacro" />
-  <!-- initial position for simulations (Mock Hardware, Gazebo) -->
-  <xacro:arg name="initial_positions_file" default="$(find kortex_description)/config/initial_positions.yaml"/>
-  <!-- convert to property to use substitution in function -->
-  <xacro:property name="initial_positions_file" default="$(arg initial_positions_file)"/>
-  <!-- create link fixed to the "world" -->
-  <link name="world" />
-  <xacro:load_robot
-    parent="world"
-    arm="$(arg arm)"
-    gripper="$(arg gripper)"
-    gripper_joint_name="$(arg gripper_joint_name)"
-    gripper_max_velocity="$(arg gripper_max_velocity)"
-    gripper_max_force="$(arg gripper_max_force)"
-    dof="$(arg dof)"
-    vision="$(arg vision)"
-    robot_ip="$(arg robot_ip)"
-    username="$(arg username)"
-    password="$(arg password)"
-    port="$(arg port)"
-    port_realtime="$(arg port_realtime)"
-    session_inactivity_timeout_ms="$(arg session_inactivity_timeout_ms)"
-    connection_inactivity_timeout_ms="$(arg connection_inactivity_timeout_ms)"
-    use_internal_bus_gripper_comm="$(arg use_internal_bus_gripper_comm)"
-    prefix="$(arg prefix)"
-    use_fake_hardware="$(arg use_fake_hardware)"
-    fake_sensor_commands="$(arg fake_sensor_commands)"
-    sim_gazebo="$(arg sim_gazebo)"
-    sim_isaac="$(arg sim_isaac)"
-    initial_positions="${xacro.load_yaml(initial_positions_file)}"
-    moveit_active="$(arg moveit_active)">
-    <origin xyz="0 0 0" rpy="0 0 0" />  <!-- position robot in the world -->
-  </xacro:load_robot>
-  <xacro:if value="$(arg sim_gazebo)">
-    <!-- Gazebo plugins -->
-    <gazebo reference="world">
-    </gazebo>
-    <gazebo>
-      <plugin filename="gz_ros2_control-system" name="gz_ros2_control::GazeboSimROS2ControlPlugin">
-        <parameters>$(arg simulation_controllers)</parameters>
-        <controller_manager_node_name>$(arg prefix)controller_manager</controller_manager_node_name>
-      </plugin>
-      <plugin filename="gz-sim-sensors-system" name="gz::sim::systems::Sensors">
-        <render_engine>$(arg gazebo_renderer)</render_engine>
-      </plugin>
-    </gazebo>
-    <gazebo reference="camera_color_frame">
-      <sensor name="camera_sensor" type="rgbd_camera">
-        <camera>
-          <horizontal_fov>1.047</horizontal_fov>
-          <image>
-            <width>$(arg camera_width)</width>
-            <height>$(arg camera_height)</height>
-            <format>RGB_INT8</format>
-          </image>
-          <clip>
-            <near>0.1</near>
-            <far>5</far>
-          </clip>
-          <distortion>
-            <k1>0.0</k1>
-            <k2>0.0</k2>
-            <k3>0.0</k3>
-            <p1>0.0</p1>
-            <p2>0.0</p2>
-            <center>0.5 0.5</center>
-          </distortion>
-          <lens>
-            <intrinsics>
-              <fx>554.25469</fx>
-              <fy>554.25469</fy>
-              <cx>320.5</cx>
-              <cy>240.5</cy>
-              <s>0</s>
-            </intrinsics>
-            <!-- These need to match the intrinsics above or
-            Gazebo will default to different default values -->
-            <projection>
-              <p_fx>554.25469</p_fx>
-              <p_fy>554.25469</p_fy>
-              <p_cx>320.5</p_cx>
-              <p_cy>240.5</p_cy>
-              <tx>0</tx>
-              <ty>0</ty>
-            </projection>
-          </lens>
-          <noise>
-            <type>gaussian</type>
-            <mean>0</mean>
-            <stddev>0.00</stddev>
-          </noise>
-          <depth_camera>
+  <robot name="$(arg name)">
+    <!-- Arguments -->
+    <xacro:arg name="prefix" default="" />
+    <xacro:arg name="arm" default="NO_ARM_TYPE_DEFINED" />
+    <xacro:arg name="dof" default="7" />
+    <xacro:arg name="vision" default="false" />
+    <xacro:arg name="robot_ip" default="192.168.11.11" />
+    <xacro:arg name="username" default="admin" />
+    <xacro:arg name="password" default="admin" />
+    <xacro:arg name="port" default="10000" />
+    <xacro:arg name="port_realtime" default="10001" />
+    <xacro:arg name="session_inactivity_timeout_ms" default="60000" />
+    <xacro:arg name="connection_inactivity_timeout_ms" default="2000" />
+    <xacro:arg name="gripper" default="" />
+    <xacro:arg name="gripper_joint_name" default="finger_joint" />
+    <xacro:arg name="gripper_max_velocity" default="100.0" />
+    <xacro:arg name="gripper_max_force" default="100.0" />
+    <xacro:arg name="use_internal_bus_gripper_comm" default="false" />
+    <xacro:arg name="use_fake_hardware" default="false" />
+    <xacro:arg name="fake_sensor_commands" default="false" />
+    <xacro:arg name="sim_gazebo" default="false" />
+    <xacro:arg name="sim_isaac" default="false" />
+    <xacro:arg name="gazebo_renderer" default="ogre"/>
+    <xacro:arg name="camera_width" default="640"/>
+    <xacro:arg name="camera_height" default="480"/>
+    <xacro:arg name="camera_fps" default="6"/>
+    <xacro:arg name="simulation_controllers" default="$(find kortex_description)/arm/$(arg arm)/$(arg dof)dof/config/ros2_controllers.yaml" />
+    <xacro:arg name="moveit_active" default="false"/>
+    <!-- import main macro -->
+    <xacro:include filename="$(find kortex_description)/robots/kortex_robot.xacro" />
+    <!-- initial position for simulations (Mock Hardware, Gazebo) -->
+    <xacro:arg name="initial_positions_file" default="$(find kortex_description)/config/initial_positions.yaml"/>
+    <!-- convert to property to use substitution in function -->
+    <xacro:property name="initial_positions_file" default="$(arg initial_positions_file)"/>
+    <!-- create link fixed to the "world" -->
+    <link name="world" />
+    <xacro:load_robot
+      parent="world"
+      arm="$(arg arm)"
+      gripper="$(arg gripper)"
+      gripper_joint_name="$(arg gripper_joint_name)"
+      gripper_max_velocity="$(arg gripper_max_velocity)"
+      gripper_max_force="$(arg gripper_max_force)"
+      dof="$(arg dof)"
+      vision="$(arg vision)"
+      robot_ip="$(arg robot_ip)"
+      username="$(arg username)"
+      password="$(arg password)"
+      port="$(arg port)"
+      port_realtime="$(arg port_realtime)"
+      session_inactivity_timeout_ms="$(arg session_inactivity_timeout_ms)"
+      connection_inactivity_timeout_ms="$(arg connection_inactivity_timeout_ms)"
+      use_internal_bus_gripper_comm="$(arg use_internal_bus_gripper_comm)"
+      prefix="$(arg prefix)"
+      use_fake_hardware="$(arg use_fake_hardware)"
+      fake_sensor_commands="$(arg fake_sensor_commands)"
+      sim_gazebo="$(arg sim_gazebo)"
+      sim_isaac="$(arg sim_isaac)"
+      initial_positions="${xacro.load_yaml(initial_positions_file)}"
+      moveit_active="$(arg moveit_active)">
+      <origin xyz="0 0 0" rpy="0 0 0" />  <!-- position robot in the world -->
+    </xacro:load_robot>
+    <xacro:if value="$(arg sim_gazebo)">
+      <!-- Gazebo plugins -->
+      <gazebo reference="world">
+      </gazebo>
+      <gazebo>
+        <plugin filename="gz_ros2_control-system" name="gz_ros2_control::GazeboSimROS2ControlPlugin">
+          <parameters>$(arg simulation_controllers)</parameters>
+          <controller_manager_node_name>$(arg prefix)controller_manager</controller_manager_node_name>
+        </plugin>
+        <plugin filename="gz-sim-sensors-system" name="gz::sim::systems::Sensors">
+          <render_engine>$(arg gazebo_renderer)</render_engine>
+        </plugin>
+      </gazebo>
+      <gazebo reference="camera_color_frame">
+        <sensor name="camera_sensor" type="rgbd_camera">
+          <camera>
+            <horizontal_fov>1.047</horizontal_fov>
+            <image>
+              <width>$(arg camera_width)</width>
+              <height>$(arg camera_height)</height>
+              <format>RGB_INT8</format>
+            </image>
             <clip>
-              <near>0.25</near>
+              <near>0.1</near>
               <far>5</far>
             </clip>
-          </depth_camera>
-          <optical_frame_id>color_optical_frame</optical_frame_id>
-        </camera>
-        <gz_frame_id>camera_color_frame</gz_frame_id>
-        <always_on>1</always_on>
-        <update_rate>$(arg camera_fps)</update_rate>
-        <visualize>true</visualize>
-        <topic>wrist_mounted_camera</topic>
-        <enable_metrics>false</enable_metrics>
-      </sensor>
-    </gazebo>
-  </xacro:if>
+            <distortion>
+              <k1>0.0</k1>
+              <k2>0.0</k2>
+              <k3>0.0</k3>
+              <p1>0.0</p1>
+              <p2>0.0</p2>
+              <center>0.5 0.5</center>
+            </distortion>
+            <lens>
+              <intrinsics>
+                <fx>554.25469</fx>
+                <fy>554.25469</fy>
+                <cx>320.5</cx>
+                <cy>240.5</cy>
+                <s>0</s>
+              </intrinsics>
+              <!-- These need to match the intrinsics above or
+              Gazebo will default to different default values -->
+              <projection>
+                <p_fx>554.25469</p_fx>
+                <p_fy>554.25469</p_fy>
+                <p_cx>320.5</p_cx>
+                <p_cy>240.5</p_cy>
+                <tx>0</tx>
+                <ty>0</ty>
+              </projection>
+            </lens>
+            <noise>
+              <type>gaussian</type>
+              <mean>0</mean>
+              <stddev>0.00</stddev>
+            </noise>
+            <depth_camera>
+              <clip>
+                <near>0.25</near>
+                <far>5</far>
+              </clip>
+            </depth_camera>
+            <optical_frame_id>color_optical_frame</optical_frame_id>
+          </camera>
+          <gz_frame_id>camera_color_frame</gz_frame_id>
+          <always_on>1</always_on>
+          <update_rate>$(arg camera_fps)</update_rate>
+          <visualize>true</visualize>
+          <topic>wrist_mounted_camera</topic>
+          <enable_metrics>false</enable_metrics>
+        </sensor>
+      </gazebo>
+    </xacro:if>
+  </robot>
 </robot>
