Commit message: 加入夹爪

File: src/table_plate_demo/urdf/kinova_gen3_fixed.urdf (robot description, URDF)
Before this commit: robot kinova_gen3, 11 links, 10 joints
Links:
- added link dummy_link
- added link gripper_base_link, mass 0.1395; collision mesh filename=file:///home/ubuntu/DishBot/install/kortex_description/shar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; visual mesh filename=file:///home/ubuntu/DishBot/install/kortex_description/shar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
- added link left_finger_dist_link, mass 0.010748; collision mesh filename=file:///home/ubuntu/DishBot/install/kortex_description/shar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; visual mesh filename=file:///home/ubuntu/DishBot/install/kortex_description/shar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
- added link left_finger_prox_link, mass 0.018385; collision mesh filename=file:///home/ubuntu/DishBot/install/kortex_description/shar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; visual mesh filename=file:///home/ubuntu/DishBot/install/kortex_description/shar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
- added link right_finger_dist_link, mass 0.010748; collision mesh filename=file:///home/ubuntu/DishBot/install/kortex_description/shar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; visual mesh filename=file:///home/ubuntu/DishBot/install/kortex_description/shar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
- added link right_finger_prox_link, mass 0.018385; collision mesh filename=file:///home/ubuntu/DishBot/install/kortex_description/shar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; visual mesh filename=file:///home/ubuntu/DishBot/install/kortex_description/shar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
Joints:
- added joint dummy_joint: type fixed, parent end_effector_link, child dummy_link, origin xyz=0 0 0 rpy=0 0 0
- added joint gripper_base_joint: type fixed, parent dummy_link, child gripper_base_link, origin xyz=0 0 0 rpy=0 0 0, axis 0 0 0
- added joint left_finger_bottom_joint: type revolute, parent gripper_base_link, child left_finger_prox_link, origin xyz=0 0.0305 0.070003 rpy=0 1.5708 0, axis 0 0 1, limit lower=-0.96 upper=0.09 effort=10 velocity=0.6
- added joint left_finger_tip_joint: type revolute, parent left_finger_prox_link, child left_finger_dist_link, origin xyz=-0.045636 -0.020423 6.9901E-05 rpy=0 0 0, axis 0 0 -1, limit lower=-0.50 upper=0.21 effort=1000 velocity=1000
- added joint right_finger_bottom_joint: type revolute, parent gripper_base_link, child right_finger_prox_link, origin xyz=0 -0.030501 0.070003 rpy=0 1.5708 0, axis 0 0 1, limit lower=-0.09 upper=0.96 effort=10 velocity=0.6
- added joint right_finger_tip_joint: type revolute, parent right_finger_prox_link, child right_finger_dist_link, origin xyz=-0.045636 0.020423 0 rpy=0 0 0, axis 0 0 1, limit lower=-0.50 upper=0.21 effort=1000 velocity=1000
- joint tool_frame_joint: origin xyz=0 0 0 rpy=0 0 0 -> xyz=0 0 0.130 rpy=0 0 1.57079632679; parent end_effector_link -> dummy_link
